Commit message: added diff_slam.launch for launching headless gazebo with gmapping

File: urdf/diff.xacro (robot description, xacro)
@@ -121,7 +121,35 @@
   <joint name="baseToLidar" type="fixed">
     <axis xyz="0 1 0"/>
-    <origin xyz="0 ${base_length*0.6/2} ${base_height/2 + lidar_height/2}" rpy="0 0 ${PI/2}"/>
+    <origin xyz="0 0 ${base_height/2 + lidar_height/2 + 0.03}" rpy="0 0 ${PI/2}"/>
     <parent link="base_link"/>
     <child link="lidar"/>
+  </joint>
+  <link name="lidar_support">
+    <xacro:property name="lidar_support_height" value="0.03"/>
+    <xacro:property name="lidar_support_radius" value="${lidar_radius/2.0}"/>
+    <visual>
+      <geometry>
+        <cylinder length="${lidar_support_height}" radius="${lidar_support_radius}"/>
+      </geometry>
+      <material name="dark"/>
+    </visual>
+    <collision>
+      <geometry>
+        <cylinder length="0.03" radius="${lidar_support_radius}"/>
+      </geometry>
+    </collision>
+    <inertial>
+      <xacro:property name="lidar_support_mass" value="0.05"/>
+      <mass value="${lidar_support_mass}"/>
+      <inertia ixx="${1/12 * lidar_support_mass * (3*lidar_support_radius**2 + lidar_support_height**2)}" ixy="0.0" ixz="0.0"
+                    iyy="${1/12 * lidar_support_mass * (3*lidar_support_radius**2 + lidar_support_height**2)}" iyz="0.0"
+                         izz="${1/2 * lidar_support_mass * lidar_support_radius**2}"/>
+    </inertial>
+  </link>
+  <joint name="baseToLidarSupport" type="fixed">
+    <axis xyz="0 1 0"/>
+    <origin xyz="0 0 ${base_height/2 + lidar_support_height/2}" rpy="0 0 ${PI/2}"/>
+    <parent link="base_link"/>
+    <child link="lidar_support"/>
   </joint>
   <xacro:property name="camera_size" value="0.02" />
